File: boards/busunit/busunit.brd (EAGLE design)
At the start: 78 x 50 mm, 21 parts, among them J1 RJ11, J2 RJ11, U1 STM32F030F4, U2 SN65HVD233D

Commit message: Minor modifications, images of board & schema included
Parts:
- moved LC0 17.3 mm to (45.7, 22.9)
- moved LC1 17.3 mm to (45.7, 5.59)
Connections:
- net LOADCELL_DT0: now also U1.11; no longer U1.10
- net LOADCELL_DT1: now also U1.10; no longer U1.11
Routing:
- net LOADCELL_DT1: track 26.7 -> 22.1 mm
- net LOADCELL_DT0: track 22.1 -> 25.2 mm
- net GND: track 195.3 -> 193.8 mm
Changed lines of the file:
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@@
 <attribute name="PROD_ID" value="VREG-08170" x="5.588" y="20.447" size="1.778" layer="27" display="off"/>
 </element>
-<element name="LC0" library="SparkFun-Connectors" package="1X04" value="" x="45.72" y="5.588" rot="R90">
+<element name="LC1" library="SparkFun-Connectors" package="1X04" value="" x="45.72" y="5.588" rot="R90">
 <attribute name="PROD_ID" value="CONN-09696" x="45.72" y="5.588" size="1.778" layer="27" rot="R90" display="off"/>
 </element>
-<element name="LC1" library="SparkFun-Connectors" package="1X04" value="" x="45.72" y="22.86" rot="R90">
+<element name="LC0" library="SparkFun-Connectors" package="1X04" value="" x="45.72" y="22.86" rot="R90">
 <attribute name="PROD_ID" value="CONN-09696" x="45.72" y="22.86" size="1.778" layer="27" rot="R90" display="off"/>
 </element>
@@
 <contactref element="C1" pad="2"/>
 <contactref element="C2" pad="2"/>
+<contactref element="LC0" pad="4"/>
 <contactref element="LC1" pad="4"/>
-<contactref element="LC0" pad="4"/>
 <contactref element="J5" pad="1"/>
 <contactref element="J5" pad="2"/>
@@
 <wire x1="8.89" y1="4.6355" x2="9.144" y2="4.826" width="0.254" layer="1"/>
 <wire x1="6.6675" y1="4.6355" x2="6.604" y2="4.826" width="0.254" layer="1"/>
-<wire x1="11.938" y1="18.058" x2="12.065" y2="19.3675" width="0.254" layer="1"/>
 <wire x1="21.2725" y1="16.51" x2="21.28" y2="16.2528" width="0.254" layer="1"/>
 <wire x1="4.039" y1="11.327" x2="4.064" y2="11.327" width="0.6096" layer="1"/>
@@
 <contactref element="J1" pad="2"/>
 <contactref element="J2" pad="2"/>
-<wire x1="34.6075" y1="38.1" x2="34.71699375" y2="38.020365625" width="0.254" layer="1"/>
+<wire x1="34.6075" y1="38.1" x2="34.71699375" y2="38.020365625" width="0" layer="19" extent="1-16"/>
 <wire x1="33.02" y1="34.925" x2="33.02" y2="35.687" width="0.6096" layer="1"/>
 <wire x1="33.02" y1="34.925" x2="32.9798" y2="34.1344" width="0.6096" layer="1"/>
@@
 <contactref element="U3" pad="4"/>
 <contactref element="C2" pad="1"/>
+<contactref element="LC0" pad="1"/>
 <contactref element="LC1" pad="1"/>
-<contactref element="LC0" pad="1"/>
 <contactref element="J4" pad="1"/>
 <contactref element="J4" pad="2"/>
@@
 <wire x1="9.906" y1="32.766" x2="10.16" y2="33.02" width="0.3048" layer="1"/>
 <wire x1="10.16" y1="33.02" x2="10.922" y2="33.02" width="0.3048" layer="1"/>
-<wire x1="10.922" y1="33.02" x2="11.176" y2="32.766" width="0.3048" layer="1"/>
-<wire x1="11.176" y1="32.766" x2="11.938" y2="32.766" width="0.3048" layer="1"/>
-<wire x1="11.938" y1="32.766" x2="12.192" y2="32.512" width="0.3048" layer="1"/>
+<wire x1="10.922" y1="33.02" x2="11.176" y2="32.893" width="0.3048" layer="1"/>
+<wire x1="11.176" y1="32.893" x2="11.811" y2="32.512" width="0.3048" layer="1"/>
+<wire x1="11.811" y1="32.512" x2="12.192" y2="32.512" width="0.3048" layer="1"/>
 <wire x1="12.192" y1="32.512" x2="14.224" y2="32.512" width="0.4064" layer="1"/>
 <wire x1="14.224" y1="32.512" x2="15.24" y2="33.528" width="0.4064" layer="1"/>
@@
 </signal>
 <signal name="LOADCELL_CLK_SHARED">
+<contactref element="LC1" pad="2"/>
 <contactref element="LC0" pad="2"/>
-<contactref element="LC1" pad="2"/>
 <contactref element="U1" pad="7"/>
 <wire x1="21.9075" y1="10.16" x2="21.93" y2="10.4172" width="0.254" layer="1"/>
@@
 <signal name="LOADCELL_DT1">
 <contactref element="LC1" pad="3"/>
-<contactref element="U1" pad="11"/>
-<wire x1="23.88" y1="16.2528" x2="25.3968" y2="16.2528" width="0.4064" layer="1"/>
-<wire x1="25.3968" y1="16.2528" x2="25.4" y2="16.256" width="0.4064" layer="1"/>
-<wire x1="25.4" y1="16.256" x2="26.416" y2="16.256" width="0.6096" layer="1"/>
-<wire x1="26.416" y1="16.256" x2="33.528" y2="23.368" width="0.6096" layer="1"/>
-<wire x1="33.528" y1="23.368" x2="39.624" y2="23.368" width="0.6096" layer="1"/>
-<wire x1="44.196" y1="27.94" x2="39.624" y2="23.368" width="0.6096" layer="1"/>
-<wire x1="45.72" y1="27.94" x2="44.196" y2="27.94" width="0.6096" layer="1"/>
+<contactref element="U1" pad="10"/>
+<wire x1="23.88" y1="10.4172" x2="24.3808" y2="10.4172" width="0.3048" layer="1"/>
+<wire x1="24.3808" y1="10.4172" x2="24.13" y2="10.414" width="0.3048" layer="1"/>
+<wire x1="24.13" y1="10.414" x2="45.466" y2="10.414" width="0.6096" layer="1"/>
+<wire x1="45.466" y1="10.414" x2="45.72" y2="10.668" width="0" layer="19" extent="1-1"/>
 </signal>
 <signal name="N$1">
@@
 <signal name="LOADCELL_DT0">
 <contactref element="LC0" pad="3"/>
-<contactref element="U1" pad="10"/>
-<wire x1="23.88" y1="10.4172" x2="24.3808" y2="10.4172" width="0.3048" layer="1"/>
-<wire x1="24.3808" y1="10.4172" x2="24.13" y2="10.414" width="0.3048" layer="1"/>
-<wire x1="24.13" y1="10.414" x2="45.466" y2="10.414" width="0.6096" layer="1"/>
-<wire x1="45.466" y1="10.414" x2="45.72" y2="10.668" width="0" layer="19" extent="1-1"/>
+<contactref element="U1" pad="11"/>
+<wire x1="23.88" y1="16.2528" x2="25.3968" y2="16.2528" width="0.4064" layer="1"/>
+<wire x1="25.3968" y1="16.2528" x2="25.4" y2="16.256" width="0.4064" layer="1"/>
+<wire x1="25.4" y1="16.256" x2="26.416" y2="16.256" width="0.6096" layer="1"/>
+<wire x1="26.416" y1="16.256" x2="33.528" y2="23.368" width="0.6096" layer="1"/>
+<wire x1="33.528" y1="23.368" x2="39.624" y2="23.368" width="0.6096" layer="1"/>
+<wire x1="44.196" y1="27.94" x2="39.624" y2="23.368" width="0.6096" layer="1"/>
+<wire x1="44.196" y1="27.94" x2="45.72" y2="27.94" width="0" layer="19" extent="1-1"/>
 </signal>
 </signals>
