File: boards/busunit/busunit.sch (EAGLE design)
At the start: 21 parts, among them J1 RJ11, J2 RJ11, U1 STM32F030F4, U2 SN65HVD233D

Commit message: Minor modifications, images of board & schema included
Connections:
- net LOADCELL_DT0: now also U1.PA5; no longer U1.PA4
- net LOADCELL_DT1: now also U1.PA4; no longer U1.PA5
Other:
- moved on the sheet: LC0, LC1
