File: boards/power_board/power_board.sch (EAGLE design)
At the start: 24 parts, among them J5 USB_A_SMT_FEMALE, J6 USB_A_SMT_FEMALE, Q2 IRFR5305, U1 YZXSTUDIO_SOLARCHARGERDEFAULT, U2 PTH08080WPTH08080W, U3 MAX2812MAX2812_SOIC8

Commit message: Minor modifications, images of board & schema included
Parts:
- R4: value 3M9 -> 3M3
- R6: value 370k -> 470k
- R7: value 820k -> 120k
- R8: value 100 -> 0
Changed lines of the file:
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@@
 <part name="R2" library="rcl" deviceset="R-EU_" device="R1206" value="1M"/>
 <part name="R3" library="rcl" deviceset="R-EU_" device="R1206" value="1M"/>
-<part name="R4" library="rcl" deviceset="R-EU_" device="R1206" value="3M9"/>
-<part name="R6" library="rcl" deviceset="R-EU_" device="R1206" value="370k"/>
+<part name="R4" library="rcl" deviceset="R-EU_" device="R1206" value="3M3"/>
+<part name="R6" library="rcl" deviceset="R-EU_" device="R1206" value="470k"/>
 <part name="F1" library="special" deviceset="FUSE" device="" value="3A"/>
 <part name="GND2" library="supply1" deviceset="GND" device=""/>
@@
 <part name="U3" library="custom_adluc" deviceset="MAX2812" device="MAX2812_SOIC8"/>
 <part name="GND8" library="supply1" deviceset="GND" device=""/>
-<part name="R8" library="rcl" deviceset="R-EU_" device="R1206" value="100"/>
-<part name="R7" library="rcl" deviceset="R-EU_" device="R1206" value="820k"/>
+<part name="R8" library="rcl" deviceset="R-EU_" device="R1206" value="0"/>
+<part name="R7" library="rcl" deviceset="R-EU_" device="R1206" value="120k"/>
 <part name="R5" library="rcl" deviceset="R-TRIMM" device="64Y" value="1M"/>
 <part name="C1" library="rcl" deviceset="CPOL-EU" device="E3.5-8" value="100u"/>
